Commit message: dockerization

File: meshes/small.urdf (robot description, URDF)
Before this commit: robot digit, 1 links, 0 joints
Links:
- link baseLink: geometry collision mesh filename=sphere.stl scale=1 1 1; visual mesh filename=sphere.stl scale=1 1 1

File: meshes/sphere_small.urdf (robot description, URDF)
Before this commit: robot urdf_robot, 1 links, 0 joints
Links:
- link base_link: geometry collision mesh filename=sphere.stl scale=1.0 1.0 1.0; visual mesh filename=sphere.stl scale=1.0 1.0 1.0
